File: LM386-toy.kicad_pcb (KiCad board)
At the start: 2 copper layers, 57.7 x 56 mm, 18 parts, among them J1 Speaker, J2 Input Volume, J3 Body Contacts, J4 LED1, J5 LED2, J6 Piezo, J7 9V, J8 ON/OFF, Q1 2N3904, U1 LM386

Commit message: fabrication v1
Parts:
- moved R3 7.63 mm to (117.3, 88.6), turned to -90 degrees
Routing:
- net Net-(C4-Pad1): track 10.00 -> 4.39 mm
- net VCC: track 61.3 -> 66.8 mm
- net /spk+: track 56.3 -> 56.9 mm
- net /touch3: vias 2 -> 3
Other:
- board text added: "v1"
